File: cpNode-Xiao.kicad_pcb (KiCad board)
At the start: 2 copper layers, 79.8 x 68.8 mm, 35 parts, among them CON2 Vout, J1 Conn_01x07_Socket, J2 Conn_01x07_Socket, J3 DCJ0202, J4 Conn_8P8C, J5 Conn_8P8C, Q1 Q_P-FET_8A_SOP-8_A04443, Q8 BSS138, Q9 BSS138, U1 XIAO-ESP32-C6, U2 MAX3491EPD+

Commit message: 3.0B
Parts:
- added D1: BAT54, Package_TO_SOT_SMD:TSOT-23, F.Cu at (125.8, 147.3)
- added R23: 120R, SPCoast:0603-RES, F.Cu at (169.6, 99.8)
- added R24: 120R, SPCoast:0603-RES, F.Cu at (174.9, 99.8)
- added TERM-RX1: Conn_01x02, SPCoast:Connector_01x02_V, F.Cu at (169.6, 105.5)
- added TERM-TX1: Conn_01x02, SPCoast:Connector_01x02_V, F.Cu at (175.3, 105.5)
- CON2: footprint Connector_PinHeader_2.54mm:PinHeader_1x04_P2.54mm_Vertical -> SPCoast:Connector_01x04_V
- DOC1: value cpNode-Xiao -> ${PROJECTNAME}
- J1, J2: footprint SPCoast:PinSocket_1x08_P2.54mm_Vertical -> SPCoast:PinSocket_1x07_P2.54mm_Vertical
- R35: value 2k2 -> 4k7
- R4: value 470 -> 330
- moved OSHW1 6.87 mm to (168.4, 91.5)
Routing:
- net Net-(TERM-TX1-Pin_1): track 75.8 -> 100.1 mm
- net Net-(U2-Y): track 67.0 -> 87.9 mm, vias 3 -> 4
- net Net-(U2-A): track 74.1 -> 92.6 mm
- net VBUS: track 22.1 -> 38.5 mm
- net Net-(TERM-RX1-Pin_1): track 83.1 -> 99.1 mm
- net Net-(D1-C): track 2.20 -> 6.81 mm
- net Net-(TERM-RX1-Pin_2): track 0.00 -> 3.39 mm
- net Net-(TERM-TX1-Pin_2): track 0.00 -> 3.21 mm
- net TXEN: track 42.1 -> 39.7 mm
- net GND: track 40.0 -> 41.3 mm
Other:
- board text added: "RS-485"
- board text added: "RS-485 Interface 3.3V"
- board text added: "RS485 Term"
- board text added: "RX"
- board text added: "TX"
- board text removed: "RS422/485 Interface 3.3V"
