File: cpNode-Xiao.kicad_sch (KiCad schematic)
At the start: 35 parts, among them CON2 Vout, J1 Conn_01x07_Socket, J2 Conn_01x07_Socket, J3 DCJ0202, J4 Conn_8P8C, J5 Conn_8P8C, Q1 Q_P-FET_8A_SOP-8_A04443, Q8 BSS138, Q9 BSS138, U1 XIAO-ESP32-C6, U2 MAX3491EPD+

Commit message: 3.0B
Parts:
- added D1: BAT54, Package_TO_SOT_SMD:TSOT-23, symbol SPCoast-eagle:DIODE-BAT54
- added R23, R24: 120R, SPCoast:0603-RES, symbol SPCoast:R
- added TERM-RX1, TERM-TX1: Conn_01x02, SPCoast:Connector_01x02_V, symbol SPCoast:Conn_01x02
- C4: footprint (none) -> SPCoast:0603-CAP
- CON2: footprint Connector_PinHeader_2.54mm:PinHeader_1x04_P2.54mm_Vertical -> SPCoast:Connector_01x04_V
- J1, J2: footprint SPCoast:PinSocket_1x08_P2.54mm_Vertical -> SPCoast:PinSocket_1x07_P2.54mm_Vertical
- J3: Voltage 5vDC -> 7.5-12VDC
- R35: value 2k2 -> 4k7
- R4: value 470 -> 330
Connections:
- net VBUS: now also D1.1 (A)
- net at J4.6, J5.6, RS485-3.1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: now also R23.2
- net at J4.3, J5.3, RS485-3.2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: now also TERM-RX1.1 (Pin_1)
- net at J4.4, J5.4, RS485-3.3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: now also R24.2
- net at J4.5, J5.5, RS485-3.4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: now also TERM-TX1.1 (Pin_1)
- net at LED2.2 (A), R5.2: now also D1.3 (C)
- new net: R24.1, TERM-TX1.2 (Pin_2)
- new net: R23.1, TERM-RX1.2 (Pin_2)
Other:
- note added: "RS485 Termination"
- title: cpNode-Xiao -> cpNode Xiao
- moved on the sheet: I2C1, I2CLED64, Q8, Q9, R21, R22, R8, R9
